File: PCBs/crosses-wired-3x5.kicad_pcb (KiCad board)
At the start: 2 copper layers, 165.1 x 115.1 mm, 81 parts, among them J1 Conn_01x14_Pin, J2 Conn_01x04_Socket, J3 Conn_01x14_Pin, J4 Conn_01x04_Socket

Commit message: Add OSH logos
Parts:
- added REF**: OSHW-Logo_5.7x6mm_SilkScreen, Symbol:OSHW-Logo_5.7x6mm_SilkScreen, B.Cu at (245.1, 149.5)
- added REF**: OSHW-Logo_5.7x6mm_SilkScreen, Symbol:OSHW-Logo_5.7x6mm_SilkScreen, B.Cu at (118.6, 149.7)
