File: PCBs/crosses-wired-3x6.kicad_pcb (KiCad board)
At the start: 2 copper layers, 165.1 x 133.6 mm, 93 parts, among them J1 Conn_01x14_Pin, J2 Conn_01x04_Socket, J3 Conn_01x14_Pin, J4 Conn_01x04_Socket

Commit message: Add OSH logos
Parts:
- added REF**: OSHW-Logo_5.7x6mm_SilkScreen, Symbol:OSHW-Logo_5.7x6mm_SilkScreen, B.Cu at (171.2, 200.3)
- added REF**: OSHW-Logo_5.7x6mm_SilkScreen, Symbol:OSHW-Logo_5.7x6mm_SilkScreen, B.Cu at (191.6, 200.5)
