File: PCBs/crosses-wired-thumb-cluster.kicad_pcb (KiCad board)
At the start: 2 copper layers, 126.8 x 111 mm, 42 parts, among them J1 Conn_01x06_Socket, J2 Conn_01x06_Socket, J4 Conn_01x14_Pin, J5 Conn_01x14_Pin, P1 TYPE-C-31-M-12 USB, P2 TYPE-C-31-M-12 USB, U1 supermini nrf / nice nano v2, U2 supermini nrf / nice nano v2

Commit message: Add OSH logos
Parts:
- added REF**: OSHW-Logo_5.7x6mm_SilkScreen, Symbol:OSHW-Logo_5.7x6mm_SilkScreen, F.Cu at (112.2, 125.5)
- added REF**: OSHW-Logo_5.7x6mm_SilkScreen, Symbol:OSHW-Logo_5.7x6mm_SilkScreen, F.Cu at (203.7, 156.0)
